Commit message: Add files via upload
Version de base

File: src/eurobot_description/gazebo/gazebo_control.xacro (robot description, xacro)
@@ -9,6 +9,6 @@
       <odometry_rate>20.0</odometry_rate>
       <robot_base_frame>base_footprint</robot_base_frame>
-      <publish_odom>false</publish_odom>
-      <publish_odom_tf>false</publish_odom_tf>
+      <publish_odom>true</publish_odom>
+      <publish_odom_tf>true</publish_odom_tf>
     </plugin>
   </gazebo>

File: src/eurobot_description/urdf/LiDAR.xacro (robot description, xacro)
@@ -26,6 +26,7 @@
             </xacro:inertial_cylinder>
         </link>
+        <!-- Simulation du LiDAR -->
         <gazebo reference='LiDAR_link'>
-            <!-- <material>Gazebo/Yellow</material> -->
+            <material>Gazebo/Yellow</material>
             <sensor name="laser" type="ray">
                 <pose> 0 0 0 0 0 0 </pose>
